File: Hardware reference/FRISTACK_IOT/FRISTACK_IOT.kicad_sch (KiCad schematic)
At the start: 56 parts, among them J2 MEM2075-00-140-01-A, J4 Conn_01x13_Socket, J5 Conn_01x13_Socket, J6 Conn_01x02_Pin, U3 TPS62840DLCR, U4 ESP32-C6-MINI-1-H4, U5 SN65HVD232, Y1 32.768 kHz

Commit message: FRISTACK_IOT_v2
Second version of iot board
Parts:
- removed TWAI1: Conn_01x04_Pin, Connector_JST:JST_PH_S4B-PH-K_1x04_P2.00mm_Horizontal, symbol Connector:Conn_01x04_Pin
- renumbered C22 to C10, C8 to C11, C13 to C12, C14 to C13, C16 to C14, C17 to C15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
Other:
- moved on the sheet: D1
