File: Hardware reference/FRISTACK_CORE/FRISTACK_CORE.kicad_sch (KiCad schematic)
At the start: 86 parts, among them J1 Conn_01x13_Socket, J2 USB_C_Receptacle_USB2.0_16P, J3 Conn_01x13_Socket, J6 JTAG_PIN_HEADER, SW1 SW_DIP_x01, SW2 SW_DIP_x01, U1 USBLC6-2SC6, U2 MCP73871-2CC, U3 TPS62840DLCR, U4 ESP32-S3-MINI-1U, U5 FSUSB42MUX, U6 SN65HVD232, Y1 32.768 kHz

Commit message: Changes to Core and Sensor Node
Parts:
- C27: footprint Capacitor_SMD:C_0402_1005Metric -> Capacitor_SMD:C_0603_1608Metric
- J6: footprint Connector_PinHeader_2.54mm:PinHeader_1x02_P2.54mm_Vertical -> Connector_PinHeader_2.54mm:PinHeader_1x02_P2.54mm_Horizontal
- R12: value 20k -> 25k
- R15: value 2k -> 15k
Changed lines of the file:
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@@
 			)
 		)
-		(property "Datasheet" "~"
+		(property "Datasheet" "C13564"
 			(at 132.08 135.89 0)
 			(effects
@@
 			)
 		)
-		(property "Footprint" "Capacitor_SMD:C_0402_1005Metric"
+		(property "Footprint" "Capacitor_SMD:C_0603_1608Metric"
 			(at 359.1052 43.18 0)
 			(effects
@@
 			)
 		)
-		(property "Value" "2k"
+		(property "Value" "15k"
 			(at 106.68 121.9199 0)
 			(effects
@@
 			)
 		)
-		(property "Footprint" "Connector_PinHeader_2.54mm:PinHeader_1x02_P2.54mm_Vertical"
+		(property "Footprint" "Connector_PinHeader_2.54mm:PinHeader_1x02_P2.54mm_Horizontal"
 			(at 384.81 129.54 0)
 			(effects
@@
 			)
 		)
-		(property "Value" "20k"
+		(property "Value" "25k"
 			(at 99.06 129.5399 0)
 			(effects
@@
 			)
 		)
-		(property "Datasheet" "DFE201612E"
+		(property "Datasheet" "DFE201612E-2R2M=P2"
 			(at 231.14 33.02 0)
 			(effects
